File: ecad/usbkvm/usb_kvm.kicad_pcb (KiCad board)
At the start: 4 copper layers, 18 x 43 mm, 44 parts, among them J1 USB_C_Receptacle, J2 USB_B_Micro, J3 USB3_A, U1 RP2040, U2 W25Q128JVS, U3 MIC5504-3.3YM5, U4 SL2.1A, Y1 ABM8-272-T3

Commit message: Good enough to release.
Parts:
- removed JP1: SolderJumper_2_Open, Jumper:SolderJumper-2_P1.3mm_Open_RoundedPad1.0x1.5mm
- removed R3: 20k, Resistor_SMD:R_0402_1005Metric_Pad0.72x0.64mm_HandSolder
- removed TP_GND1, TP_GP26, TP_GP27, TP_SWCLK1, TP_SWD1: TestPoint, TestPoint:TestPoint_Pad_1.0x1.0mm
- added C1: 1u, Capacitor_SMD:C_0402_1005Metric_Pad0.74x0.62mm_HandSolder, F.Cu at (97.8, 68.3)
- added C11: 1u, Capacitor_SMD:C_0402_1005Metric_Pad0.74x0.62mm_HandSolder, F.Cu at (94.6, 74.7)
- added C16: 100n, Capacitor_SMD:C_0402_1005Metric_Pad0.74x0.62mm_HandSolder, F.Cu at (106.2, 72.1)
- added R14: 27.4, Resistor_SMD:R_0402_1005Metric_Pad0.72x0.64mm_HandSolder, F.Cu at (94.6, 72.6)
- added TP1: TestPoint, TestPoint:TestPoint_THTPad_D1.0mm_Drill0.5mm, F.Cu at (94.6, 70.0)
- added TP10: TestPoint, TestPoint:TestPoint_Pad_1.5x1.5mm, B.Cu at (101.7, 64.0)
- added TP11: TestPoint, TestPoint:TestPoint_Pad_1.5x1.5mm, B.Cu at (102.2, 66.5)
- added TP12: TestPoint, TestPoint:TestPoint_THTPad_D1.0mm_Drill0.5mm, F.Cu at (94.9, 67.7)
- added TP2: TestPoint, TestPoint:TestPoint_Pad_1.5x1.5mm, B.Cu at (101.7, 76.5)
- added TP3: TestPoint, TestPoint:TestPoint_Pad_1.5x1.5mm, B.Cu at (101.7, 73.9)
- added TP4: TestPoint, TestPoint:TestPoint_Pad_1.5x1.5mm, B.Cu at (101.7, 71.4)
- added TP5: TestPoint, TestPoint:TestPoint_THTPad_D1.0mm_Drill0.5mm, F.Cu at (105.5, 82.0)
- added TP6: TestPoint, TestPoint:TestPoint_THTPad_D1.0mm_Drill0.5mm, F.Cu at (105.2, 80.0)
- added TP7: TestPoint, TestPoint:TestPoint_THTPad_D1.0mm_Drill0.5mm, F.Cu at (99.0, 55.4)
- added TP9: TestPoint, TestPoint:TestPoint_Pad_1.5x1.5mm, B.Cu at (103.9, 61.5)
- added U5: W25Q128JVS, Package_SO:SOIC-8_5.23x5.23mm_P1.27mm, F.Cu at (99.3, 80.8)
- C17: value 10u -> 1u
- C18, C19, C20: value 10u -> 100n
- R10: value 20k -> 10k
- R11: value 10k -> 5.1k
- R6: value 100 -> 10k
- R7: value 100 -> 27.4
- R8, R9: value 22 -> 27.4
- U4: value SL2.1A -> RP2040; footprint Package_SO:SOP-16_3.9x9.9mm_P1.27mm -> Package_DFN_QFN:QFN-56-1EP_7x7mm_P0.4mm_EP3.2x3.2mm
- moved C6 22.0 mm to (106.2, 61.7), turned to 90 degrees
- moved C2 21.0 mm to (105.7, 51.1), turned to -90 degrees
- moved C14 20.7 mm to (100.6, 58.4)
- moved R6 19.5 mm to (103.5, 58.7)
- moved C12 18.4 mm to (106.0, 67.8), turned to 90 degrees
- moved C15 17.3 mm to (106.2, 64.0)
- moved C3 16.7 mm to (100.8, 54.6), turned to 90 degrees
- moved C19 16.7 mm to (94.0, 82.3), turned to 90 degrees
- moved C9 16.1 mm to (98.6, 58.4), turned to 90 degrees
- moved U1 15.0 mm to (101.4, 63.6), turned to 90 degrees
- moved C10 14.9 mm to (99.6, 58.4)
- moved R2 14.4 mm to (104.4, 57.7), turned to 180 degrees
- moved Y1 14.1 mm to (104.2, 54.6)
- moved C8 12.6 mm to (96.0, 61.6), turned to 180 degrees
- moved R11 12.6 mm to (106.2, 76.7)
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Connections:
- C18 pad 1: VBUS -> Net-(U4-VREG_VOUT)
- C19 pad 1: Net-(U4-VDD3) -> +3.3V
- C20 pad 1: Net-(U4-VDD18) -> +3.3V
- J3 pad 2: /USB_REC_N -> unconnected-(J3-D--Pad2)
- J3 pad 3: /USB_REC_P -> unconnected-(J3-D+-Pad3)
- R10 pad 2: Net-(U1-GPIO1) -> /GUEST_VBUS_EN
- R11 pad 1: Net-(U1-GPIO1) -> /GUEST_VBUS_EN
- R12 pad 1: Net-(U1-GPIO8) -> Net-(U1-GPIO27_ADC1)
- R4 pad 1: /USB_RP_P -> /USB_P
- R5 pad 1: /USB_RP_N -> /USB_N
- R6 pad 1: /RP_CLK_OUT -> /GUEST_RUN
- R6 pad 2: /SL2_XIN -> GND
- R7 pad 1: GND -> Net-(U4-USB_DP)
- R7 pad 2: /SL2_XIN -> /USB_MIC_P
- R8 pad 1: Net-(U1-GPIO2) -> /USB_MIC_N
- R8 pad 2: /USB_MIC_N -> Net-(U1-GPIO29_ADC3)
- R9 pad 1: Net-(U1-GPIO3) -> Net-(U1-GPIO28_ADC2)
- U1 pad 11: Net-(U1-GPIO8) -> unconnected-(U1-GPIO8-Pad11)
- U1 pad 15: +3.3V -> unconnected-(U1-GPIO12-Pad15)
- U1 pad 16: GND -> unconnected-(U1-GPIO13-Pad16)
- U1 pad 17: GND -> unconnected-(U1-GPIO14-Pad17)
- U1 pad 18: GND -> /GUEST_VBUS_EN
- U1 pad 2: unconnected-(U1-GPIO0-Pad2) -> /HTG_CLK
- U1 pad 26: unconnected-(U1-RUN-Pad26) -> +3.3V
- U1 pad 3: Net-(U1-GPIO1) -> /HTG_D0
- U1 pad 30: unconnected-(U1-GPIO19-Pad30) -> /GUEST_RUN
- U1 pad 32: unconnected-(U1-GPIO21-Pad32) -> /RP_CLK_OUT
- U1 pad 35: /RP_CLK_OUT -> unconnected-(U1-GPIO23-Pad35)
- U1 pad 38: Net-(U1-GPIO26_ADC0) -> unconnected-(U1-GPIO26_ADC0-Pad38)
- U1 pad 4: Net-(U1-GPIO2) -> /HTG_D1
- U1 pad 40: unconnected-(U1-GPIO28_ADC2-Pad40) -> Net-(U1-GPIO28_ADC2)
- U1 pad 41: unconnected-(U1-GPIO29_ADC3-Pad41) -> Net-(U1-GPIO29_ADC3)
- U1 pad 5: Net-(U1-GPIO3) -> /HTD_D2
- U1 pad 6: unconnected-(U1-GPIO4-Pad6) -> /HTG_D3
- U1 pad 7: unconnected-(U1-GPIO5-Pad7) -> /GTH_CLK
- U1 pad 8: unconnected-(U1-GPIO6-Pad8) -> /GTH_D0
- U1 pad 9: unconnected-(U1-GPIO7-Pad9) -> /GUEST_WATCHDOG
- U4 pad 1: /USB_RP_N -> +3.3V
- U4 pad 10: /USB_P -> +3.3V
- U4 pad 11: VBUS -> unconnected-(U4-GPIO8-Pad11)
- U4 pad 12: GND -> unconnected-(U4-GPIO9-Pad12)
- U4 pad 13: Net-(U4-VDD3) -> unconnected-(U4-GPIO10-Pad13)
- U4 pad 14: Net-(U4-VDD18) -> unconnected-(U4-GPIO11-Pad14)
- U4 pad 16: /SL2_XIN -> unconnected-(U4-GPIO13-Pad16)
- U4 pad 2: /USB_RP_P -> unconnected-(U4-GPIO0-Pad2)
- U4 pad 7: /USB_REC_N -> unconnected-(U4-GPIO5-Pad7)
- U4 pad 8: /USB_REC_P -> unconnected-(U4-GPIO6-Pad8)
- U4 pad 9: /USB_N -> unconnected-(U4-GPIO7-Pad9)
Routing:
- net GND: track 73.7 -> 159.8 mm, vias 23 -> 30
- net +3.3V: track 83.9 -> 135.3 mm, vias 13 -> 3
- net Net-(J2-VBUS): track 3.63 -> 34.6 mm, vias 0 -> 2
- net Net-(U4-VREG_VOUT): track 0.00 -> 30.0 mm, vias 0 -> 3
- net /GUEST_RUN: track 0.00 -> 23.6 mm, vias 0 -> 2
- net /USB_REC_P: track 21.7 -> 0.00 mm
- net /USB_REC_N: track 21.4 -> 0.00 mm
- net Net-(U1-GPIO28_ADC2): track 0.00 -> 19.0 mm, vias 0 -> 2
- net Net-(U1-GPIO27_ADC1): track 4.05 -> 22.4 mm, vias 1 -> 2
- net /GUEST_VBUS_EN: track 0.00 -> 14.9 mm, vias 0 -> 2
- net Net-(U4-QSPI_SS): track 0.00 -> 14.4 mm
- net Net-(U1-GPIO29_ADC3): track 0.00 -> 13.9 mm, vias 0 -> 2
- net Net-(U1-QSPI_SS): track 28.3 -> 14.6 mm, vias 2 -> 0
- net /SWD: track 15.0 -> 1.69 mm
- net Net-(U1-QSPI_SD0): track 21.1 -> 7.88 mm, vias 2 -> 0
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- removed copper zone on In2.Cu, net +3.3V
- removed copper zone on In1.Cu, net GND
- removed copper zone on In2.Cu, net GND
- removed copper zone on In2.Cu, net VBUS
Other:
- board size 18 x 43 mm -> 20 x 43 mm
- copper layers 4 -> 2
- board text added: "3.3V"
- board text added: "DN"
- board text added: "DP"
- board text added: "G"
- board text added: "GND"
- board text added: "GS"
- board text added: "HS"
- board text added: "PIO USB"
- board text added: "SCK"
- board text added: "SWD"
- board text added: "Targeting: OSHPARK 2 Layer Prototype Service"
- board text added: "USB 3.0 Only (Capture card)"
- board text added: "USB 3.0 one way"
- board text removed: "SWCLK GND SWDIO"
- board text removed: "Targeting OshPark 4 Layer Stackup"
- board text removed: "USB 3.0 Capture"
- board text removed: "USB KVM V1.0"
- board text removed: "github.com/ Kytezign/USBKVM"
