File: ecad/usbkvm/usb_kvm.kicad_sch (KiCad schematic)
At the start: 44 parts, among them J1 USB_C_Receptacle, J2 USB_B_Micro, J3 USB3_A, U1 RP2040, U2 W25Q128JVS, U3 MIC5504-3.3YM5, U4 SL2.1A, Y1 ABM8-272-T3

Commit message: Good enough to release.
Parts:
- removed JP1: SolderJumper_2_Open, symbol Jumper:SolderJumper_2_Open
- removed R3: 20k, Resistor_SMD:R_0402_1005Metric_Pad0.72x0.64mm_HandSolder, symbol Device:R
- removed TP_GP26, TP_GP27: TestPoint, TestPoint:TestPoint_Pad_1.0x1.0mm, symbol Connector:TestPoint
- removed U4: SL2.1A, Package_SO:SOP-16_3.9x9.9mm_P1.27mm, symbol proj_lib:SL2.1A
- added C1, C11: 1u, Capacitor_SMD:C_0402_1005Metric_Pad0.74x0.62mm_HandSolder, symbol Device:C
- added C16: 100n, Capacitor_SMD:C_0402_1005Metric_Pad0.74x0.62mm_HandSolder, symbol Device:C
- added R14: 27.4, Resistor_SMD:R_0402_1005Metric_Pad0.72x0.64mm_HandSolder, symbol Device:R
- added TP1, TP12, TP5, TP6, TP7: TestPoint, TestPoint:TestPoint_THTPad_D1.0mm_Drill0.5mm, symbol Connector:TestPoint
- added TP2, TP3, TP4: TestPoint, TestPoint:TestPoint_Pad_1.5x1.5mm, symbol Connector:TestPoint
- added U4: RP2040, Package_DFN_QFN:QFN-56-1EP_7x7mm_P0.4mm_EP3.2x3.2mm, symbol MCU_RaspberryPi:RP2040
- added U5: W25Q128JVS, Package_SO:SOIC-8_5.23x5.23mm_P1.27mm, symbol Memory_Flash:W25Q128JVS
- C17: value 10u -> 1u
- C18, C19, C20: value 10u -> 100n
- R10: value 20k -> 10k
- R11: value 10k -> 5.1k
- R12: now not fitted
- R6: value 100 -> 10k
- R7: value 100 -> 27.4
- R8, R9: value 22 -> 27.4; now not fitted
- TP10: renamed from TP_GND1; footprint TestPoint:TestPoint_Pad_1.0x1.0mm -> TestPoint:TestPoint_Pad_1.5x1.5mm
- TP11: renamed from TP_SWCLK1; footprint TestPoint:TestPoint_Pad_1.0x1.0mm -> TestPoint:TestPoint_Pad_1.5x1.5mm
- TP9: renamed from TP_SWD1; footprint TestPoint:TestPoint_Pad_1.0x1.0mm -> TestPoint:TestPoint_Pad_1.5x1.5mm
Connections:
- net USB_RP_N is gone; now on net USB_N: R5.1
- net USB_RP_P is gone; now on net USB_P: R4.1
- net +3.3V: now also C19.1, C20.1, U1.26 (RUN), C1.2, TP7.1, U4.1 (IOVDD), U4.10 (IOVDD), U4.22 (IOVDD), U4.33 (IOVDD), U4.42 (IOVDD), U4.43 (ADC_AVDD), U4.44 (VREG_IN), U4.48 (USB_VDD), U4.49 (IOVDD), U5.8 (VCC); no longer U1.15 (GPIO12)
- net GND: now also R6.2, C1.1, C11.2, C16.2, TP1.1, TP3.1, TP5.1, U4.19 (TESTEN), U4.57 (GND), U5.4 (GND); no longer R7.1, U1.16 (GPIO13), U1.17 (GPIO14), U1.18 (GPIO15)
- net RP_CLK_OUT: now also U1.32 (GPIO21), U4.20 (XIN); no longer R6.1, U1.35 (GPIO23)
- net USB_MIC_N: now also R8.1, R14.2; no longer R8.2
- net USB_MIC_P: now also R7.2
- net VBUS: no longer C18.1
- net HTG_D1: now reaches U1.4 (GPIO2)
- net HTG_D1: now also U4.39 (GPIO27_ADC1); no longer R8.1
- net at R9.1: now also U1.40 (GPIO28_ADC2); no longer U1.5 (GPIO3)
- net GUEST_VBUS_EN: now reaches R10.2, R11.1
- net GUEST_VBUS_EN: now also U1.18 (GPIO15), U4.18 (GPIO15); no longer U1.3 (GPIO1)
- net at U1.56 (QSPI_SS), U2.1 (~{CS}): now also TP12.1
- net at U1.39 (GPIO27_ADC1): now also R12.1
- net at U1.11 (GPIO8): no longer R12.1
- net HTG_CLK: now reaches U1.2 (GPIO0)
- net HTG_CLK: now also U4.41 (GPIO29_ADC3)
- net GUEST_RUN: now reaches U1.30 (GPIO19)
- net GUEST_RUN: now also R6.1, U4.26 (RUN)
- net at U1.41 (GPIO29_ADC3): now also R8.2
- net HTG_D3: now reaches U1.6 (GPIO4)
- net HTG_D3: now also U4.37 (GPIO25)
- net GTH_CLK: now reaches U1.7 (GPIO5)
- net GTH_CLK: now also U4.36 (GPIO24)
- net GTH_D0: now reaches U1.8 (GPIO6)
- net GTH_D0: now also U4.35 (GPIO23)
- net GUEST_WATCHDOG: now reaches U1.9 (GPIO7)
- net GUEST_WATCHDOG: now also U4.34 (GPIO22)
- removed net SL2_XIN: R6.2, R7.2
- net USB_REC_N: no longer names the net of J3.2 (D-)
- net USB_REC_P: no longer names the net of J3.3 (D+)
- new net: TP4.1, U4.25 (SWD)
- new net: R7.1, U4.47 (USB_DP)
- new net: TP6.1, U4.56 (QSPI_SS), U5.1 (~{CS})
- new net: U4.55 (QSPI_SD1), U5.2 (DO(IO1))
- new net: U4.54 (QSPI_SD2), U5.3 (IO2)
- new net: U4.53 (QSPI_SD0), U5.5 (DI(IO0))
- new net: U4.52 (QSPI_SCLK), U5.6 (CLK)
- new net: U4.51 (QSPI_SD3), U5.7 (IO3)
- new net: C11.1, C16.1, C18.1, U4.23 (DVDD), U4.45 (VREG_VOUT), U4.50 (DVDD)
- new net: TP2.1, U4.24 (SWCLK)
- new net: R14.1, U4.46 (USB_DM)
- new net HTD_D2: U1.5 (GPIO3), U4.38 (GPIO26_ADC0)
- new net HTG_D0: U1.3 (GPIO1), U4.40 (GPIO28_ADC2)
- no-connect marks 9 -> 10
Other:
- note added: "GPIO Function: CLOCK GPOUT0 (see clock_gpio_init)"
- note removed: "GPIO12-15: Version 0x1"
- note removed: "Near 3.3V decoupling."
- moved on the sheet: C17, J2, R10, R11
